Commit message: correct stls and urdf

File: src/palletizing_amr/urdf/palletizing_amr.urdf (robot description, URDF)
Before this commit: robot palletizing_amr, 10 links, 9 joints
Joints:
- joint prismatic_forklift: origin xyz=-0.000092 0.685419 -0.069984 rpy=0 0 0 -> xyz=-0.00058 0.72555 -0.18250 rpy=0 0 0
- joint revolute_wheel_FLI: origin xyz=-0.138142 1.083424 -0.127388 rpy=0 0 0 -> xyz=-0.13815 1.07475 -0.26250 rpy=0 0 0
- joint revolute_wheel_FLO: origin xyz=-0.233142 1.083424 -0.127388 rpy=0 0 0 -> xyz=-0.23315 1.07475 -0.26250 rpy=0 0 0
- joint revolute_wheel_FRI: origin xyz=0.141858 1.083424 -0.127388 rpy=0 0 0 -> xyz=0.14185 1.07475 -0.26250 rpy=0 0 0
- joint revolute_wheel_FRO: origin xyz=0.226858 1.083424 -0.127388 rpy=0 0 0 -> xyz=0.22685 1.07475 -0.26250 rpy=0 0 0
- joint revolute_wheel_ML1: origin xyz=-0.175642 -0.094276 -0.114388 rpy=0 0 0 -> xyz=-0.17565 -0.10295 -0.24950 rpy=0 0 0
- joint revolute_wheel_ML2: origin xyz=-0.175642 -0.004276 -0.114388 rpy=0 0 0 -> xyz=-0.17565 -0.01295 -0.24950 rpy=0 0 0
- joint revolute_wheel_MR1: origin xyz=0.176958 -0.094276 -0.114388 rpy=0 0 0 -> xyz=0.17695 -0.10295 -0.24950 rpy=0 0 0
- joint revolute_wheel_MR2: origin xyz=0.176938 -0.004286 -0.114388 rpy=0 0 0 -> xyz=0.17693 -0.01296 -0.24950 rpy=0 0 0

Commit message: updates 2

File: src/palletizing_amr/urdf/palletizing_amr.urdf (robot description, URDF)
Before this commit: robot palletizing_amr, 10 links, 9 joints
Links:
- added link base_footprint
- added link camera_link, mass 0.05; collision box size=0.05 0.08 0.05; visual box size=0.05 0.08 0.05
- added link lidar_link, mass 0.1; collision cylinder length=0.03 radius=0.04; visual cylinder length=0.03 radius=0.04
Joints:
- added joint base_footprint_joint: type fixed, parent base_footprint, child base_link, origin xyz=0 0 0 rpy=0 0 0
- added joint camera_joint: type fixed, parent base_link, child camera_link, origin xyz=0.22 0.0 0.16 rpy=0 0 0
- added joint lidar_joint: type fixed, parent base_link, child lidar_link, origin xyz=0.18 0.0 0.22 rpy=0 0 0
- joint revolute_wheel_FLI: origin xyz=-0.13815 1.07475 -0.26250 rpy=0 0 0 -> xyz=-0.13758 0.34920 -0.08000 rpy=0 0 0; parent base_link -> forklift
- joint revolute_wheel_FLO: origin xyz=-0.23315 1.07475 -0.26250 rpy=0 0 0 -> xyz=-0.23258 0.34920 -0.08000 rpy=0 0 0; parent base_link -> forklift
- joint revolute_wheel_FRI: origin xyz=0.14185 1.07475 -0.26250 rpy=0 0 0 -> xyz=0.14243 0.34920 -0.08000 rpy=0 0 0; parent base_link -> forklift
- joint revolute_wheel_FRO: origin xyz=0.22685 1.07475 -0.26250 rpy=0 0 0 -> xyz=0.22743 0.34920 -0.08000 rpy=0 0 0; parent base_link -> forklift
- joint revolute_wheel_ML1: limit (none) -> effort=100 velocity=15
- joint revolute_wheel_ML2: limit (none) -> effort=100 velocity=15
- joint revolute_wheel_MR1: limit (none) -> effort=100 velocity=15
- joint revolute_wheel_MR2: limit (none) -> effort=100 velocity=15

Commit message: camera working and line added but not a line follower yet

File: src/palletizing_amr/urdf/palletizing_amr.urdf (robot description, URDF)
Before this commit: robot palletizing_amr, 13 links, 12 joints
Links:
- added link wheel_CL, mass 0.12; collision cylinder length=0.02 radius=0.028
- added link wheel_CR, mass 0.12; collision cylinder length=0.02 radius=0.028
- added link wheel_stabL, mass 0.12; collision cylinder length=0.02 radius=0.028
- added link wheel_stabR, mass 0.12; collision cylinder length=0.02 radius=0.028
- link base_link: mass 18.0 -> 160.0
- link camera_link: geometry collision box size=0.005 0.008 0.005; visual box size=0.005 0.008 0.005
- link forklift: geometry collision mesh filename=package://palletizing_amr/meshes/forklift.stl scale=0.001 0.001 0.001; visual mesh filename=package://palletizing_amr/meshes/forklift.stl scale=0.001 0.001 0.001
- link lidar_link: geometry collision cylinder length=0.003 radius=0.01; visual cylinder length=0.003 radius=0.01
Joints:
- added joint revolute_wheel_CL: type continuous, parent base_link, child wheel_CL, origin xyz=-0.15 0.3 -0.2495 rpy=0 0 0, axis 1 0 0
- added joint revolute_wheel_CR: type continuous, parent base_link, child wheel_CR, origin xyz=0.15 0.3 -0.2495 rpy=0 0 0, axis 1 0 0
- added joint revolute_wheel_stabL: type continuous, parent base_link, child wheel_stabL, origin xyz=-0.22 0.68 -0.2495 rpy=0 0 0, axis 1 0 0
- added joint revolute_wheel_stabR: type continuous, parent base_link, child wheel_stabR, origin xyz=0.22 0.68 -0.2495 rpy=0 0 0, axis 1 0 0
- joint camera_joint: origin xyz=0.22 0.0 0.16 rpy=0 0 0 -> xyz=0.0 -0.205 0.24 rpy=0 1.5708 0
- joint lidar_joint: origin xyz=0.18 0.0 0.22 rpy=0 0 0 -> xyz=0.0 -0.19 0.248 rpy=0 0 0
- joint prismatic_forklift: limit lower=0.0 upper=0.20 effort=1000 velocity=0.5 -> lower=0.0 upper=0.20 effort=5000 velocity=0.5
- joint revolute_wheel_ML1: limit effort=100 velocity=15 -> effort=1500 velocity=15
- joint revolute_wheel_ML2: limit effort=100 velocity=15 -> effort=1500 velocity=15
- joint revolute_wheel_MR1: limit effort=100 velocity=15 -> effort=1500 velocity=15
- joint revolute_wheel_MR2: limit effort=100 velocity=15 -> effort=1500 velocity=15

Commit message: localized pallet models

File: src/palletizing_amr/urdf/palletizing_amr.urdf (robot description, URDF)
Before this commit: robot palletizing_amr, 17 links, 16 joints
Joints:
- joint camera_joint: origin xyz=0.0 -0.205 0.24 rpy=0 1.5708 0 -> xyz=0.0 -0.205 0.24 rpy=0 0.3854 -1.5708
